File: kicad_files/raphael.kicad_sch (KiCad schematic)
At the start: 345 parts, among them J1 A1001WR-S-04P, J2 TYPE-C-31-M-12, Q1 AO3401A, Q2 2N7002, Q3 2N7002, SW1 K2-1187SQ-A4SW-06, SW10 Mechanical_Switch, SW11 Mechanical_Switch, SW12 Mechanical_Switch, SW13 Mechanical_Switch, SW14 Mechanical_Switch, SW15 Mechanical_Switch, SW16 Mechanical_Switch, SW17 Mechanical_Switch, SW18 Mechanical_Switch, SW19 Mechanical_Switch, SW2 Mechanical_Switch, SW20 Mechanical_Switch, SW21 Mechanical_Switch, SW22 Mechanical_Switch, SW23 Mechanical_Switch, SW24 Mechanical_Switch, SW25 Mechanical_Switch, SW26 Mechanical_Switch, SW27 Mechanical_Switch, SW28 Mechanical_Switch, SW29 Mechanical_Switch, SW3 Mechanical_Switch, SW30 Mechanical_Switch, SW31 Mechanical_Switch, SW32 Mechanical_Switch, SW33 Mechanical_Switch, SW34 Mechanical_Switch, SW35 Mechanical_Switch, SW36 Mechanical_Switch, SW37 Mechanical_Switch, SW38 Mechanical_Switch, SW39 Mechanical_Switch, SW4 Mechanical_Switch, SW40 Mechanical_Switch, SW41 Mechanical_Switch, SW42 Mechanical_Switch, SW43 Mechanical_Switch, SW44 Mechanical_Switch, SW45 Mechanical_Switch, SW46 Mechanical_Switch, SW47 Mechanical_Switch, SW48 Mechanical_Switch, SW49 Mechanical_Switch, SW5 Mechanical_Switch, SW50 Mechanical_Switch, SW51 Mechanical_Switch, SW52 Mechanical_Switch, SW53 Mechanical_Switch, SW54 Mechanical_Switch, SW55 Mechanical_Switch, SW56 Mechanical_Switch, SW57 Mechanical_Switch, SW58 Mechanical_Switch, SW59 Mechanical_Switch, SW6 Mechanical_Switch, SW60 Mechanical_Switch, SW61 Mechanical_Switch, SW62 Mechanical_Switch, SW63 Mechanical_Switch, SW64 Mechanical_Switch, SW65 Mechanical_Switch, SW66 Mechanical_Switch, SW67 Mechanical_Switch, SW68 Mechanical_Switch, SW69 Mechanical_Switch, SW7 Mechanical_Switch, SW70 Mechanical_Switch, SW71 Mechanical_Switch, SW72 Mechanical_Switch, SW73 Mechanical_Switch, SW74 Mechanical_Switch, SW75 Mechanical_Switch, SW76 Mechanical_Switch, SW77 Mechanical_Switch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

Commit message: Update submodules
Parts:
- R75: value (none) -> 100R; footprint (none) -> Resistor_SMD:R_0805_2012Metric
- R76: value (none) -> 10k; footprint (none) -> Resistor_SMD:R_0805_2012Metric
- U4: value (none) -> BL24C256A-SFRC; footprint (none) -> acheron_Components:TSSOP-8_4.4x3mm_P0.65mm
Changed lines of the file:
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@@
       (effects (font (size 1.27 1.27)) (justify right))
     )
-    (property "Value" "" (id 1) (at 149.86 1022.9849 0)
+    (property "Value" "10k" (id 1) (at 149.86 1022.9849 0)
       (effects (font (size 1.27 1.27)) (justify right))
     )
-    (property "Footprint" "" (id 2) (at 151.765 1022.35 0)
+    (property "Footprint" "Resistor_SMD:R_0805_2012Metric" (id 2) (at 151.765 1022.35 0)
       (effects (font (size 1.27 1.27)) hide)
     )
@@
     (in_bom yes) (on_board yes) (fields_autoplaced)
     (property "Reference" "R75" (id 0) (at 145.415 1009.65 90))
-    (property "Value" "" (id 1) (at 145.415 1012.19 90))
-    (property "Footprint" "" (id 2) (at 145.415 1016 0)
+    (property "Value" "100R" (id 1) (at 145.415 1012.19 90))
+    (property "Footprint" "Resistor_SMD:R_0805_2012Metric" (id 2) (at 145.415 1016 0)
       (effects (font (size 1.27 1.27)) hide)
     )
@@
     (pin "2")
     (pin "6")
-    (pin "3")
-    (pin "4")
-    (pin "5")
   )
   (symbol (lib_id "Device:D_Small") (at 352.425 462.915 270) (unit 1)
@@
     (in_bom yes) (on_board yes)
     (property "Reference" "U4" (id 0) (at 53.975 50.8 0))
-    (property "Value" "" (id 1) (at 47.625 53.34 0))
-    (property "Footprint" "" (id 2) (at 57.15 60.96 0)
+    (property "Value" "BL24C256A-SFRC" (id 1) (at 47.625 53.34 0))
+    (property "Footprint" "acheron_Components:TSSOP-8_4.4x3mm_P0.65mm" (id 2) (at 57.15 60.96 0)
       (effects (font (size 1.27 1.27)) hide)
     )
@@
       (effects (font (size 1.27 1.27)) hide)
     )
-    (pin "1")
-    (pin "2")
-    (pin "6")
     (pin "3")
     (pin "4")
